File: analog-keypad-16-keys/analog-keypad-16-keys.kicad_sch (KiCad schematic)
At the start: 34 parts, among them J1 Conn_01x03_Pin, SW1 SW_Push_Dual, SW10 SW_Push_Dual, SW11 SW_Push_Dual, SW12 SW_Push_Dual, SW13 SW_Push_Dual, SW14 SW_Push_Dual, SW15 SW_Push_Dual, SW16 SW_Push_Dual, SW2 SW_Push_Dual, SW3 SW_Push_Dual, SW4 SW_Push_Dual, SW5 SW_Push_Dual, SW6 SW_Push_Dual, SW7 SW_Push_Dual, SW8 SW_Push_Dual, SW9 SW_Push_Dual

Commit message: schematic finished, PCB started
schematic finished, PCB started
Parts:
- removed J1: Conn_01x03_Pin, symbol Connector:Conn_01x03_Pin
- added D1, D2: LED, LED_THT:LED_D5.0mm_Clear, symbol Device:LED
- added J1: Conn_01x04_Pin, Connector_PinHeader_2.54mm:PinHeader_1x04_P2.54mm_Vertical, symbol Connector:Conn_01x04_Pin
- added R18, R19: 2k2, Resistor_SMD:R_0805_2012Metric, symbol Device:R
- R1: value R -> 2k7; footprint (none) -> Resistor_SMD:R_0805_2012Metric
- R10: value R -> 56k; footprint (none) -> Resistor_SMD:R_0805_2012Metric
- R11: value R -> 120k; footprint (none) -> Resistor_SMD:R_0805_2012Metric
- R12: value R -> 6k8; footprint (none) -> Resistor_SMD:R_0805_2012Metric
- R13: value R -> 33k; footprint (none) -> Resistor_SMD:R_0805_2012Metric
- R14: value R -> 68k; footprint (none) -> Resistor_SMD:R_0805_2012Metric
- R15: value R -> 133k; footprint (none) -> Resistor_SMD:R_0805_2012Metric
- R16: value R -> 8k2; footprint (none) -> Resistor_SMD:R_0805_2012Metric
- R17, R6: value R -> 47k; footprint (none) -> Resistor_SMD:R_0805_2012Metric
- R2: value R -> 10k; footprint (none) -> Resistor_SMD:R_0805_2012Metric
- R3: value R -> 39k; footprint (none) -> Resistor_SMD:R_0805_2012Metric
- R4: value R -> 82k; footprint (none) -> Resistor_SMD:R_0805_2012Metric
- R5: value R -> 15k; footprint (none) -> Resistor_SMD:R_0805_2012Metric
- R7: value R -> 100k; footprint (none) -> Resistor_SMD:R_0805_2012Metric
- R8: value R -> 4k7; footprint (none) -> Resistor_SMD:R_0805_2012Metric
- R9: value R -> 22k; footprint (none) -> Resistor_SMD:R_0805_2012Metric
- SW1, SW10, SW11, SW12, SW13, SW14, SW15, SW16, SW2, SW3, SW4, SW5, SW6, SW7, SW8, SW9: footprint (none) -> Button_Switch_THT:SW_PUSH_6mm
Connections:
- net at SW4.1: now also R4.2
- net Signal: now reaches SW4.2
- net Signal: now also R17.1, SW1.2, SW10.2, SW11.2, SW12.2, SW13.2, SW14.2, SW15.2, SW16.2, SW2.2, SW3.2, SW5.2, SW6.2, SW7.2, SW8.2, SW9.2, J1.2 (Pin_2)
- net at SW11.1: now also R10.2
- net VCC: now reaches R15.1
- net VCC: now also R1.1, R10.1, R11.1, R12.1, R13.1, R14.1, R16.1, R2.1, R3.1, R4.1, R5.1, R6.1, R7.1, R8.1, R9.1, D1.2 (A), J1.1 (Pin_1)
- net at R15.2: now also SW16.1
- net at R13.2: now also SW14.1
- net at R14.2: now also SW15.1
- net at R11.2: now also SW12.1
- net GND: now reaches R17.2
- net GND: now also D2.1 (K), J1.4 (Pin_4)
- net at R9.2: now also SW10.1
- net at SW3.1: now also R3.2
- net at R7.2: now also SW8.1
- net at R2.2: now also SW2.1
- net at SW6.1: now also R5.2
- net at SW13.1: now also R16.2
- net at R8.2: now also SW5.1
- net at R12.2: now also SW9.1
- net at R6.2: now also SW7.1
- net at R1.2: now also SW1.1
- new net: D1.1 (K), R18.2
- new net: D2.2 (A), R19.1
- new net LEDs: J1.3 (Pin_3), R18.1, R19.2
Other:
- moved on the sheet: R1, R10, R11, R12, R13, R14, R15, R16, R17, R2, R3, R4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
