File: analog-keypad-16-keys/analog-keypad-16-keys.kicad_pcb (KiCad board)
At the start: 2 copper layers, 60 x 70 mm, 38 parts, among them J1 Conn_01x04_Pin, SW1 SW_Push_Dual, SW10 SW_Push_Dual, SW11 SW_Push_Dual, SW12 SW_Push_Dual, SW13 SW_Push_Dual, SW14 SW_Push_Dual, SW15 SW_Push_Dual, SW16 SW_Push_Dual, SW2 SW_Push_Dual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

Commit message: Started PCB layout
Parts:
- moved R19 119.1 mm to (146.4, 41.7), turned to -90 degrees
- moved R13 117.9 mm to (146.3, 60.2)
- moved R14 115.5 mm to (146.6, 74.9)
- moved R16 114.9 mm to (146.9, 46.0)
- moved R15 110.0 mm to (146.7, 90.0)
- moved R12 108.1 mm to (131.9, 46.1)
- moved R9 101.0 mm to (131.8, 60.1)
- moved R18 100.8 mm to (127.6, 41.6), turned to 90 degrees
- moved R10 99.5 mm to (132.1, 74.9)
- moved D2 99.2 mm to (140.4, 40.1)
- moved R11 98.7 mm to (131.6, 89.9)
- moved D1 97.6 mm to (131.1, 40.1)
- moved R5 93.2 mm to (117.0, 60.1), turned to 180 degrees
- moved R6 90.4 mm to (117.2, 75.0)
- moved R8 89.6 mm to (116.9, 46.3)
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Routing:
- net Signal: track 0.00 -> 264.6 mm
- net VCC: track 0.00 -> 75.5 mm
- net GND: track 0.00 -> 30.7 mm
Other:
- outline, holes or cut-outs redrawn

Commit message: finished PCB
Parts:
- turned R1 to 0 degrees
- turned R2 to 0 degrees
- turned R3 to 0 degrees
- turned R4 to 0 degrees
Routing:
- net VCC: track 75.5 -> 307.5 mm, vias 0 -> 1
- net LEDs: track 0.00 -> 45.0 mm
- net GND: track 30.7 -> 1.34 mm, vias 0 -> 1
- net Net-(R2-Pad2): track 0.00 -> 11.1 mm
- net Net-(R5-Pad2): track 0.00 -> 11.0 mm
- net Net-(R14-Pad2): track 0.00 -> 11.0 mm
- net Net-(R10-Pad2): track 0.00 -> 11.0 mm
- net Net-(R9-Pad2): track 0.00 -> 11.0 mm
- net Net-(R13-Pad2): track 0.00 -> 11.0 mm
- net Net-(R3-Pad2): track 0.00 -> 10.9 mm
- net Net-(R6-Pad2): track 0.00 -> 10.9 mm
- net Net-(R11-Pad2): track 0.00 -> 10.8 mm
- net Net-(R7-Pad2): track 0.00 -> 10.7 mm
- net Net-(R15-Pad2): track 0.00 -> 10.6 mm
- net Net-(R4-Pad2): track 0.00 -> 10.6 mm
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- added copper zone on B.Cu, net GND
Other:
- board text added: "1 - F1"
- board text added: "10 - #7"
- board text added: "11 - #8"
- board text added: "12 - #9"
- board text added: "13 - F4"
- board text added: "14 - ESC"
- board text added: "15 - #0"
- board text added: "16 - ENTER"
- board text added: "2 - #1"
- board text added: "3 - #2"
- board text added: "4 - #3"
- board text added: "5 - F2"
- board text added: "6 - #4"
- board text added: "7 - #5"
- board text added: "8 - #6"
- board text added: "9 - F3"
- board text added: "LED 1"
- board text added: "LED 2"
- board text added: "VCC|Signal|LEDs|GND"
